File: udb-s.kicad_pcb (KiCad board)
At the start: 4 copper layers, 40 x 9 mm, 11 parts, among them J1 TYPE-C-31-M-12, J2 78171-0004, U1 TPD4E05U06DQAR

Commit message: Redesigned
Parts:
- removed D1: ESD5Z5V0, Diode_SMD:D_SOD-523
- removed F1: SMD0805-050-16V, Fuse:Fuse_1206_3216Metric
- removed G***: LOGO, locallib:UnifiedLogo
- removed U1: TPD4E05U06DQAR, acheron_Components:USON-10_2.5x1.0mm_P0.5mm
- added F2: 1A PTC, Fuse:Fuse_0402_1005Metric, F.Cu at (129.8, 92.5)
- added U2: USBLC6-2SC6, Package_TO_SOT_SMD:SOT-23-6, F.Cu at (129.8, 94.8)
- FB1: value GZ2012D601TF -> 100R @ 100MHz; footprint Inductor_SMD:L_0805_2012Metric -> Inductor_SMD:L_0603_1608Metric
- J1: footprint locallib:HRO-TYPE-C-31-M-12-Assembly -> Connector_USB:USB_C_Receptacle_HRO_TYPE-C-31-M-12
- J2: value 78171-0004 -> SM04B-SRSS; footprint locallib:PicoEZMate-Reinforced-Lite -> Connector_JST:JST_SH_SM04B-SRSS-TB_1x04-1MP_P1.00mm_Horizontal
- moved FB1 4.80 mm to (133.2, 97.3)
- moved J1 3.65 mm to (139.1, 92.8)
- moved R1 2.34 mm to (129.8, 98.0), turned to 180 degrees
- moved R2 1.09 mm to (129.8, 97.0), turned to 180 degrees
- moved J2 0.28 mm to (122.0, 96.2)
Connections:
- J1 pad A5: Net-(J1-PadA5) -> Net-(J1-CC1)
- R1 pad 1: GND -> Net-(J1-CC1)
- R1 pad 2: Net-(J1-PadA5) -> GND
Routing:
- net D-: track 49.5 -> 27.0 mm, vias 5 -> 0
- net D+: track 49.6 -> 27.3 mm, vias 5 -> 0
- net Net-(J1-CC1): track 0.00 -> 16.0 mm, vias 0 -> 2
- net Net-(J1-PadA5): track 12.8 -> 0.00 mm, vias 2 -> 0
- net GND: track 0.43 -> 8.44 mm, vias 6 -> 7
- net 5V: track 9.19 -> 14.9 mm, vias 2 -> 3
- net VBUS: track 29.3 -> 24.8 mm, vias 2 -> 3
- net GNDPWR: track 10.0 -> 6.88 mm
- net Net-(J1-CC2): track 10.9 -> 9.27 mm
Other:
- board text added: "hunger solving world peace giving universal son board"
- board text removed: "USE ONLY uDB CABLES"
- board text removed: "Unified-S1 V1.1"
- board text removed: "Unified-S1 V1.1 www.unified- daughterboard.github.io"
