File: udb-s.kicad_sch (KiCad schematic)
At the start: 10 parts, among them J1 TYPE-C-31-M-12, J2 78171-0004, U1 TPD4E05U06DQAR

Commit message: Redesigned
Parts:
- removed D1: ESD5Z5V0, Diode_SMD:D_SOD-523, symbol Diode:SMF6V0A
- removed F1: SMD0805-050-16V, Fuse:Fuse_1206_3216Metric, symbol Device:Fuse
- removed FB1: GZ2012D601TF, Inductor_SMD:L_0805_2012Metric, symbol Device:FerriteBead
- removed R1, R2: 5.1k, Resistor_SMD:R_0402_1005Metric, symbol Device:R_Small
- removed U1: TPD4E05U06DQAR, acheron_Components:USON-10_2.5x1.0mm_P0.5mm, symbol acheron_Symbols:TPD4E05U06DQAR
- added F2: 1A PTC, Fuse:Fuse_0402_1005Metric, symbol Device:Polyfuse_Small
- added FB1: 100R @ 100MHz, Inductor_SMD:L_0603_1608Metric, symbol Device:FerriteBead_Small
- added R1, R2: 5.1k, Resistor_SMD:R_0402_1005Metric, symbol Device:R_Small_US
- added U2: USBLC6-2SC6, Package_TO_SOT_SMD:SOT-23-6, symbol Power_Protection:USBLC6-2SC6
- J1: footprint locallib:HRO-TYPE-C-31-M-12-Assembly -> Connector_USB:USB_C_Receptacle_HRO_TYPE-C-31-M-12
- J2: value 78171-0004 -> SM04B-SRSS; footprint locallib:PicoEZMate-Reinforced-Lite -> Connector_JST:JST_SH_SM04B-SRSS-TB_1x04-1MP_P1.00mm_Horizontal; LCSC Part Number C588524 -> C160404; Manufacturer MOLEX -> JST; Manufacturer Part Number 78171-0004 -> SM04B-SRSS-TB
Connections:
- net 5V: now also F2.2, U2.5 (VBUS)
- net D+: now also U2.3 (I/O2), U2.4 (I/O2)
- net D-: now also U2.1 (I/O1), U2.6 (I/O1)
- net GND: now also FB1.2, R1.2, R2.2, U2.2 (GND)
- net GNDPWR: now also FB1.1
- net VBUS: now also F2.1
- net at J1.A5 (CC1): now also R1.1
- net at J1.B5 (CC2): now also R2.1
Other:
- note added: "ESD"
- note removed: "USB ESD"
- moved on the sheet: J1
